File: HardWare/AS5047P/HardWare/AS5047P.kicad_sch (KiCad schematic)
At the start: 5 parts, among them J1 CONN_1x5P, J2 CONN_1x5P, U1 AS5047D

Commit message: 添加AS5047P无刷电机硬件模块设计
Parts:
- added D2: Yellow LED, LED_SMD:LED_0603_1608Metric, symbol Device:LED
- added R4: 1K, Resistor_SMD:R_0603_1608Metric, symbol Device:R_Small_US
- J1: footprint SAMTEC_ZF5S-05-02-T-WT -> 3rd_Connector_JST_SMD:CONN-SMD_1x5P-P1.0-H_WAFER-SH1.0-5PWB
- J2: footprint SAMTEC_ZF5S-06-02-T-WT -> 3rd_Connector_JST_SMD:CONN-SMD_1x6P-P1.0-H_WAFER-SH1.0-6PWB
Connections:
- net +5V: now also R4.1
- net GND: now also D2.1 (K)
- new net: D2.2 (A), R4.2
Changed lines of the file:
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@@
+    (stroke (width 0) (type default))
+  )
+  (wire (pts (xy 102.87 106.68) (xy 102.87 105.41))
     (stroke (width 0) (type default))
   )
@@
     (stroke (width 0) (type default))
   )
+  (wire (pts (xy 102.87 96.52) (xy 102.87 97.79))
+    (stroke (width 0) (type default))
+  )
   (wire (pts (xy 182.88 86.36) (xy 186.69 86.36))
     (stroke (width 0) (type default))
@@
   )
   (wire (pts (xy 180.34 115.57) (xy 186.69 115.57))
+    (stroke (width 0) (type default))
+  )
+  (wire (pts (xy 102.87 90.17) (xy 102.87 91.44))
     (stroke (width 0) (type default))
   )
@@
     )
   )
+  (symbol (lib_id "power:+5V") (at 102.87 90.17 0) (unit 1)
+    (in_bom yes) (on_board yes) (dnp no)
+    (property "Reference" "#PWR09" (at 102.87 93.98 0)
+      (effects (font (size 1.27 1.27)) hide)
+    )
+    (property "Value" "+5V" (at 102.87 85.09 90)
+      (effects (font (size 1.27 1.27)))
+    )
+    (property "Footprint" "" (at 102.87 90.17 0)
+      (effects (font (size 1.27 1.27)) hide)
+    )
+    (property "Datasheet" "" (at 102.87 90.17 0)
+      (effects (font (size 1.27 1.27)) hide)
+    )
+    (pin "1")
+    (instances
+      (project "AS5047P"
+        (path "/a1100fb3-9bb1-4a7b-859f-32d730218ced"
+          (reference "#PWR09") (unit 1)
+        )
+      )
+    )
+  )
+  (symbol (lib_id "power:GND") (at 102.87 106.68 0) (unit 1)
+    (in_bom yes) (on_board yes) (dnp no)
+    (property "Reference" "#PWR08" (at 102.87 113.03 0)
+      (effects (font (size 1.27 1.27)) hide)
+    )
+    (property "Value" "GND" (at 102.87 110.49 0)
+      (effects (font (size 1.27 1.27)))
+    )
+    (property "Footprint" "" (at 102.87 106.68 0)
+      (effects (font (size 1.27 1.27)) hide)
+    )
+    (property "Datasheet" "" (at 102.87 106.68 0)
+      (effects (font (size 1.27 1.27)) hide)
+    )
+    (pin "1")
+    (instances
+      (project "AS5047P"
+        (path "/a1100fb3-9bb1-4a7b-859f-32d730218ced"
+          (reference "#PWR08") (unit 1)
+        )
+      )
+    )
+  )
+  (symbol (lib_id "Device:LED") (at 102.87 101.6 90) (unit 1)
+    (in_bom yes) (on_board yes) (dnp no)
+    (property "Reference" "D2" (at 105.41 100.33 0)
+      (effects (font (size 1.27 1.27)) (justify right))
+    )
+    (property "Value" "Yellow LED" (at 99.06 97.79 0)
+      (effects (font (size 1.27 1.27)) (justify right))
+    )
+    (property "Footprint" "LED_SMD:LED_0603_1608Metric" (at 102.87 101.6 0)
+      (effects (font (size 1.27 1.27)) hide)
+    )
+    (property "Datasheet" "~" (at 102.87 101.6 0)
+      (effects (font (size 1.27 1.27)) hide)
+    )
+    (pin "1")
+    (pin "2")
+    (instances
+      (project "MotorKit"
+        (path "/3221bc87-9952-46a0-bacd-9685c4728da5"
+          (reference "D2") (unit 1)
+        )
+      )
+      (project "AS5047P"
+        (path "/a1100fb3-9bb1-4a7b-859f-32d730218ced"
+          (reference "D1") (unit 1)
+        )
+      )
+      (project "StepDriver"
+        (path "/e63e39d7-6ac0-4ffd-8aa3-1841a4541b55"
+          (reference "D9") (unit 1)
+        )
+      )
+    )
+  )
   (symbol (lib_id "power:+5V") (at 180.34 115.57 90) (unit 1)
     (in_bom yes) (on_board yes) (dnp no)
@@
       (effects (font (size 1.27 1.27)) (justify left))
     )
-    (property "Footprint" "SAMTEC_ZF5S-06-02-T-WT" (at 198.12 123.19 0)
+    (property "Footprint" "3rd_Connector_JST_SMD:CONN-SMD_1x6P-P1.0-H_WAFER-SH1.0-6PWB" (at 198.12 123.19 0)
       (effects (font (size 1.27 1.27)) (justify bottom) hide)
     )
@@
     )
   )
+  (symbol (lib_id "Device:R_Small_US") (at 102.87 93.98 0) (mirror y) (unit 1)
+    (in_bom yes) (on_board yes) (dnp no)
+    (property "Reference" "R4" (at 105.41 96.52 90)
+      (effects (font (size 1.27 1.27)) (justify left))
+    )
+    (property "Value" "1K" (at 105.41 93.98 90)
+      (effects (font (size 1.27 1.27)) (justify left))
+    )
+    (property "Footprint" "Resistor_SMD:R_0603_1608Metric" (at 102.87 93.98 0)
+      (effects (font (size 1.27 1.27)) hide)
+    )
+    (property "Datasheet" "~" (at 102.87 93.98 0)
+      (effects (font (size 1.27 1.27)) hide)
+    )
+    (pin "1")
+    (pin "2")
+    (instances
+      (project "MotorKit"
+        (path "/3221bc87-9952-46a0-bacd-9685c4728da5"
+          (reference "R4") (unit 1)
+        )
+      )
+      (project "AS5047P"
+        (path "/a1100fb3-9bb1-4a7b-859f-32d730218ced"
+          (reference "R1") (unit 1)
+        )
+      )
+      (project "StepDriver"
+        (path "/e63e39d7-6ac0-4ffd-8aa3-1841a4541b55"
+          (reference "R28") (unit 1)
+        )
+      )
+    )
+  )
   (symbol (lib_id "power:+5V") (at 146.05 82.55 0) (unit 1)
     (in_bom yes) (on_board yes) (dnp no)
@@
       (effects (font (size 1.27 1.27)) (justify left))
     )
-    (property "Footprint" "SAMTEC_ZF5S-05-02-T-WT" (at 195.58 101.6 0)
+    (property "Footprint" "3rd_Connector_JST_SMD:CONN-SMD_1x5P-P1.0-H_WAFER-SH1.0-5PWB" (at 195.58 101.6 0)
       (effects (font (size 1.27 1.27)) (justify bottom) hide)
     )
